File: kicad/kicad.kicad_sch (KiCad schematic)
At the start: 0 parts

Commit message: Create brushed DC motor controller baseline
Other:
- note added: "1 INPUT PROTECTION AND MOTOR SUPPLY J1: VIN_12V, PGND F1: fuse/PTC after motor current is measured D_TVS1: TVS footprint placeholder, final value TBD C_BULK1: 470uF 25V near motor connector Nets: VIN_12V, VMOTOR_12V, PGND"
- note added: "2 LOW-SIDE MOTOR SWITCH M1: small 12V brushed DC motor Q1: logic-level N-MOSFET, exact part TBD D1: flyback diode from MOTOR_SW to VMOTOR_12V R_GATE: 22 ohm start value R_PD: 100k gate pulldown Nets: PWM_GATE, MOTOR_SW, MOTOR_CURRENT_SHUNT_HI"
- note added: "3 CURRENT SENSE R_SHUNT1: 0.05 ohm 1W candidate U_ISENSE1: INA180A1 gain 20 candidate RC filter before STM32 ADC Nets: MOTOR_CURRENT_SHUNT_HI, MOTOR_CURRENT_SHUNT_LO, ISENSE_ADC, AGND"
- note added: "4 VOLTAGE AND TEMPERATURE SENSE R_VTOP1/R_VBOT1: 100k/27k candidate divider R_NTC1: 10k NTC candidate near MOSFET or motor connector RC filters near ADC pins Nets: VSENSE_ADC, TEMP_ADC, VDD_3V3, AGND"
- note added: "5 STM32 NUCLEO AND CAN U_DEV1: NUCLEO-G0B1RE header interface U_CAN1: 3.3V CAN transceiver candidate TCAN332 R_TERM1: optional 120 ohm termination jumper J_ACC1: 3.3V I2C/SPI accelerometer module header Nets: CAN_TX, CAN_RX, CANH, CANL, VDD_3V3"
- note added: "NUCLEO-G0B1RE + one-direction low-side MOSFET + shunt current sensing + CAN transceiver"
- note added: "REQUIRED TEST POINTS TP_VIN_12V, TP_VMOTOR_12V, TP_PWM_GATE, TP_MOTOR_SW, TP_SHUNT_HI, TP_SHUNT_LO, TP_ISENSE_ADC, TP_VSENSE_ADC, TP_TEMP_ADC, TP_3V3, TP_CANH, TP_CANL, TP_PGND"
- note added: "VERSION 1 SELECTED ARCHITECTURE"
- company: (none) -> Student portfolio project
- title: (none) -> Smart Brushed DC Motor Controller - Version 1
Changed lines of the file:
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@@
 	(generator_version "10.0")
 	(paper "A4")
+	(title_block
+		(title "Smart Brushed DC Motor Controller - Version 1")
+		(date "2026-07-12")
+		(rev "0.1")
+		(company "Student portfolio project")
+		(comment 1 "First-pass schematic roadmap. Replace text blocks with checked symbols before PCB layout.")
+	)
+	(text "VERSION 1 SELECTED ARCHITECTURE"
+		(at 18 18 0)
+		(effects
+			(font
+				(size 3 3)
+				(thickness 0.3)
+			)
+			(justify left)
+		)
+	)
+	(text "NUCLEO-G0B1RE + one-direction low-side MOSFET + shunt current sensing + CAN transceiver"
+		(at 18 25 0)
+		(effects
+			(font
+				(size 1.5 1.5)
+				(thickness 0.15)
+			)
+			(justify left)
+		)
+	)
+	(text "1 INPUT PROTECTION AND MOTOR SUPPLY\nJ1: VIN_12V, PGND\nF1: fuse/PTC after motor current is measured\nD_TVS1: TVS footprint placeholder, final value TBD\nC_BULK1: 470uF 25V near motor connector\nNets: VIN_12V, VMOTOR_12V, PGND"
+		(at 18 38 0)
+		(effects
+			(font
+				(size 1.27 1.27)
+				(thickness 0.15)
+			)
+			(justify left)
+		)
+	)
+	(text "2 LOW-SIDE MOTOR SWITCH\nM1: small 12V brushed DC motor\nQ1: logic-level N-MOSFET, exact part TBD\nD1: flyback diode from MOTOR_SW to VMOTOR_12V\nR_GATE: 22 ohm start value\nR_PD: 100k gate pulldown\nNets: PWM_GATE, MOTOR_SW, MOTOR_CURRENT_SHUNT_HI"
+		(at 18 72 0)
+		(effects
+			(font
+				(size 1.27 1.27)
+				(thickness 0.15)
+			)
+			(justify left)
+		)
+	)
+	(text "3 CURRENT SENSE\nR_SHUNT1: 0.05 ohm 1W candidate\nU_ISENSE1: INA180A1 gain 20 candidate\nRC filter before STM32 ADC\nNets: MOTOR_CURRENT_SHUNT_HI, MOTOR_CURRENT_SHUNT_LO, ISENSE_ADC, AGND"
+		(at 18 109 0)
+		(effects
+			(font
+				(size 1.27 1.27)
+				(thickness 0.15)
+			)
+			(justify left)
+		)
+	)
+	(text "4 VOLTAGE AND TEMPERATURE SENSE\nR_VTOP1/R_VBOT1: 100k/27k candidate divider\nR_NTC1: 10k NTC candidate near MOSFET or motor connector\nRC filters near ADC pins\nNets: VSENSE_ADC, TEMP_ADC, VDD_3V3, AGND"
+		(at 18 138 0)
+		(effects
+			(font
+				(size 1.27 1.27)
+				(thickness 0.15)
+			)
+			(justify left)
+		)
+	)
+	(text "5 STM32 NUCLEO AND CAN\nU_DEV1: NUCLEO-G0B1RE header interface\nU_CAN1: 3.3V CAN transceiver candidate TCAN332\nR_TERM1: optional 120 ohm termination jumper\nJ_ACC1: 3.3V I2C/SPI accelerometer module header\nNets: CAN_TX, CAN_RX, CANH, CANL, VDD_3V3"
+		(at 18 165 0)
+		(effects
+			(font
+				(size 1.27 1.27)
+				(thickness 0.15)
+			)
+			(justify left)
+		)
+	)
+	(text "REQUIRED TEST POINTS\nTP_VIN_12V, TP_VMOTOR_12V, TP_PWM_GATE, TP_MOTOR_SW, TP_SHUNT_HI, TP_SHUNT_LO,\nTP_ISENSE_ADC, TP_VSENSE_ADC, TP_TEMP_ADC, TP_3V3, TP_CANH, TP_CANL, TP_PGND"
+		(at 18 198 0)
+		(effects
+			(font
+				(size 1.27 1.27)
+				(thickness 0.15)
+			)
+			(justify left)
+		)
+	)
 	(sheet_instances
 		(path "/"

Commit message: Select version 1 motor electronics
Parts:
- added C1: 470uF 25V, Capacitor_THT:CP_Radial_D8.0mm_P3.50mm, symbol Device:CP
- added C2, C3: 47nF, Capacitor_SMD:C_0805_2012Metric, symbol Device:C
- added D1: 1N5822, Diode_THT:D_DO-201AD_P15.24mm_Horizontal, symbol Diode:1N5822
- added D2: SMBJ18A, Diode_SMD:D_SMB, symbol Device:D_TVS
- added F1: RXEF110, Fuse:Fuse_Littelfuse_RXEF, symbol Device:Fuse
- added J1: 12V_IN, TerminalBlock:TerminalBlock_Altech_AK300-2_P5.00mm, symbol Connector_Generic:Conn_01x02
- added J2: MOTOR_POLOLU_3039, TerminalBlock:TerminalBlock_Altech_AK300-2_P5.00mm, symbol Connector_Generic:Conn_01x02
- added J3: NUCLEO_G0B1RE_IF, Connector_PinHeader_2.54mm:PinHeader_1x09_P2.54mm_Vertical, symbol Connector_Generic:Conn_01x09
- added J4: CAN, TerminalBlock:TerminalBlock_OnShore_OSTVN03A150, symbol Connector_Generic:Conn_01x03
- added Q1: IRLZ44NPBF, Package_TO_SOT_THT:TO-220-3_Vertical, symbol Transistor_FET:IRLZ44N
- added R1: 0.05R 1%, Resistor_SMD:R_2512_6332Metric, symbol Device:R
- added R2: 22R, Resistor_SMD:R_0805_2012Metric, symbol Device:R
- added R3, R4: 100k, Resistor_SMD:R_0805_2012Metric, symbol Device:R
- added R5: 27k, Resistor_SMD:R_0805_2012Metric, symbol Device:R
- added R6: 1k, Resistor_SMD:R_0805_2012Metric, symbol Device:R
- added R7: 120R optional, Resistor_SMD:R_0805_2012Metric, symbol Device:R
- added RT1: 10k NTC, Sensor_Temperature:Thermistor_Bead, symbol Device:Thermistor_NTC
- added U1: TC4427ACPA, Package_DIP:DIP-8_W7.62mm, symbol Driver_FET:TC4427xOA
- added U2: INA180A1IDBVR, Package_TO_SOT_SMD:SOT-23-5, symbol Amplifier_Current:INA180A1
- added U3: TCAN332DR, Package_SO:SOIC-8_3.9x4.9mm_P1.27mm, symbol Interface_CAN_LIN:TCAN332
Other:
- note added: "Current, voltage, and temperature sensing"
- note added: "Input protection and motor supply"
- note added: "Low-side MOSFET motor switch"
- note added: "STM32 Nucleo, CAN, accelerometer header, and test points"
- note removed: "1 INPUT PROTECTION AND MOTOR SUPPLY J1: VIN_12V, PGND F1: fuse/PTC after motor current is measured D_TVS1: TVS footprint placeholder, final value TBD C_BULK1: 470uF 25V near motor connector Nets: VIN_12V, VMOTOR_12V, PGND"
- note removed: "2 LOW-SIDE MOTOR SWITCH M1: small 12V brushed DC motor Q1: logic-level N-MOSFET, exact part TBD D1: flyback diode from MOTOR_SW to VMOTOR_12V R_GATE: 22 ohm start value R_PD: 100k gate pulldown Nets: PWM_GATE, MOTOR_SW, MOTOR_CURRENT_SHUNT_HI"
- note removed: "3 CURRENT SENSE R_SHUNT1: 0.05 ohm 1W candidate U_ISENSE1: INA180A1 gain 20 candidate RC filter before STM32 ADC Nets: MOTOR_CURRENT_SHUNT_HI, MOTOR_CURRENT_SHUNT_LO, ISENSE_ADC, AGND"
- note removed: "4 VOLTAGE AND TEMPERATURE SENSE R_VTOP1/R_VBOT1: 100k/27k candidate divider R_NTC1: 10k NTC candidate near MOSFET or motor connector RC filters near ADC pins Nets: VSENSE_ADC, TEMP_ADC, VDD_3V3, AGND"
- note removed: "5 STM32 NUCLEO AND CAN U_DEV1: NUCLEO-G0B1RE header interface U_CAN1: 3.3V CAN transceiver candidate TCAN332 R_TERM1: optional 120 ohm termination jumper J_ACC1: 3.3V I2C/SPI accelerometer module header Nets: CAN_TX, CAN_RX, CANH, CANL, VDD_3V3"
- note removed: "NUCLEO-G0B1RE + one-direction low-side MOSFET + shunt current sensing + CAN transceiver"
- note removed: "REQUIRED TEST POINTS TP_VIN_12V, TP_VMOTOR_12V, TP_PWM_GATE, TP_MOTOR_SW, TP_SHUNT_HI, TP_SHUNT_LO, TP_ISENSE_ADC, TP_VSENSE_ADC, TP_TEMP_ADC, TP_3V3, TP_CANH, TP_CANL, TP_PGND"
- note removed: "VERSION 1 SELECTED ARCHITECTURE"

Commit message: Repair KiCad schematic symbols and current limits
Parts:
- removed C1: 470uF 25V, Capacitor_THT:CP_Radial_D8.0mm_P3.50mm, symbol Device:CP
- removed C2, C3: 47nF, Capacitor_SMD:C_0805_2012Metric, symbol Device:C
- removed D1: 1N5822, Diode_THT:D_DO-201AD_P15.24mm_Horizontal, symbol Diode:1N5822
- removed D2: SMBJ18A, Diode_SMD:D_SMB, symbol Device:D_TVS
- removed F1: RXEF110, Fuse:Fuse_Littelfuse_RXEF, symbol Device:Fuse
- removed J1: 12V_IN, TerminalBlock:TerminalBlock_Altech_AK300-2_P5.00mm, symbol Connector_Generic:Conn_01x02
- removed J2: MOTOR_POLOLU_3039, TerminalBlock:TerminalBlock_Altech_AK300-2_P5.00mm, symbol Connector_Generic:Conn_01x02
- removed J3: NUCLEO_G0B1RE_IF, Connector_PinHeader_2.54mm:PinHeader_1x09_P2.54mm_Vertical, symbol Connector_Generic:Conn_01x09
- removed J4: CAN, TerminalBlock:TerminalBlock_OnShore_OSTVN03A150, symbol Connector_Generic:Conn_01x03
- removed Q1: IRLZ44NPBF, Package_TO_SOT_THT:TO-220-3_Vertical, symbol Transistor_FET:IRLZ44N
- removed R1: 0.05R 1%, Resistor_SMD:R_2512_6332Metric, symbol Device:R
- removed R2: 22R, Resistor_SMD:R_0805_2012Metric, symbol Device:R
- removed R3, R4: 100k, Resistor_SMD:R_0805_2012Metric, symbol Device:R
- removed R5: 27k, Resistor_SMD:R_0805_2012Metric, symbol Device:R
- removed R6: 1k, Resistor_SMD:R_0805_2012Metric, symbol Device:R
- removed R7: 120R optional, Resistor_SMD:R_0805_2012Metric, symbol Device:R
- removed RT1: 10k NTC, Sensor_Temperature:Thermistor_Bead, symbol Device:Thermistor_NTC
- removed U1: TC4427ACPA, Package_DIP:DIP-8_W7.62mm, symbol Driver_FET:TC4427xOA
- removed U2: INA180A1IDBVR, Package_TO_SOT_SMD:SOT-23-5, symbol Amplifier_Current:INA180A1
- removed U3: TCAN332DR, Package_SO:SOIC-8_3.9x4.9mm_P1.27mm, symbol Interface_CAN_LIN:TCAN332
- added C1: 470uF 25V, Capacitor_THT:CP_Radial_D8.0mm_P3.50mm, symbol V1:C_V
- added C4: 100nF, Capacitor_SMD:C_0805_2012Metric, symbol V1:C_V
- added D1: 1N5822 flyback, Diode_THT:D_DO-201AD_P15.24mm_Horizontal, symbol V1:DIODE_V
- added D2: SMBJ18A TVS, Diode_SMD:D_SMB, symbol V1:DIODE_V
- added F1: RXEF110 PTC, Fuse:Fuseholder5x20_horiz_open, symbol V1:R_H
- added J1: 12V_IN, TerminalBlock:TerminalBlock_1x02_P5.00mm, symbol V1:CONN2
- added J2: MOTOR_POLOLU_3039, TerminalBlock:TerminalBlock_1x02_P5.00mm, symbol V1:CONN2
- added J3: NUCLEO_G0B1RE_IF, Connector_PinHeader_2.54mm:PinHeader_1x09_P2.54mm_Vertical, symbol V1:CONN9
- added J4: CAN, TerminalBlock:TerminalBlock_1x03_P3.50mm, symbol V1:CONN3
- added Q1: IRLZ44NPBF, Package_TO_SOT_THT:TO-220-3_Vertical, symbol V1:NMOS
- added R1: 0.05R shunt, Resistor_SMD:R_2512_6332Metric, symbol V1:R_V
- added R2: 22R gate, Resistor_SMD:R_0805_2012Metric, symbol V1:R_H
- added R3: 100k pulldown, Resistor_SMD:R_0805_2012Metric, symbol V1:R_V
- added R4: 100k, Resistor_SMD:R_0805_2012Metric, symbol V1:R_V
- added R5: 27k, Resistor_SMD:R_0805_2012Metric, symbol V1:R_V
- added R7: 120R optional, Resistor_SMD:R_0805_2012Metric, symbol V1:R_V
- added U1: TC4427ACPA, Package_DIP:DIP-8_W7.62mm, symbol V1:GATE_DRIVER
- added U2: INA180A1IDBVR, Package_TO_SOT_SMD:SOT-23-5, symbol V1:INA180
- added U3: TCAN332DR, Package_SO:SOIC-8_3.9x4.9mm_P1.27mm, symbol V1:CAN
Connections:
- net CANH: now also J4.3, R7.2, U3.6 (CANL)
- net CAN_RX: now also J3.4 (TEMP), U3.4 (RXD)
- net ISENSE_ADC: now also J3.8 (5V), R4.2, U2.1 (OUT)
- net MOTOR_CURRENT_SHUNT_HI: now also Q1.2 (S), R1.1, R1.2, U2.3 (IN-), U2.4 (IN-)
- net PWM_FROM_STM32: now also J3.9 (GND), U1.4 (IN_B)
- net VDD_5V: now also C4.2, J3.2 (ISENSE), U1.3 (GND)
- new net: R2.1, U1.7 (OUT_A)
- new net CANL: J4.1, R7.1, U3.7 (CANH)
- new net CAN_TX: J3.5 (CAN_TX), U3.1 (TXD)
- new net MOTOR_SW: J2.1, Q1.3 (D)
- new net PGND: C4.1, J1.1, J3.1 (GND), J4.2, R3.1, R3.2, U1.2 (IN_A), U1.6 (GND), U3.3 (GND)
- new net PWM_GATE: Q1.1 (G), R2.2
- new net TEMP_ADC: J3.6 (CAN_RX)
- new net VDD_3V3: J3.3 (VSENSE), U2.5 (GND), U3.2 (GND)
- new net VIN_12V: F1.1, J1.2
- new net VMOTOR_12V: D1.1 (K), D1.2 (A), F1.2, J2.2, U2.2 (GND)
- new net VSENSE_ADC: J3.7 (3V3), R4.1, R5.1, R5.2
Other:
- note added: "Motor switch, flyback, shunt, and gate drive"
- note added: "Sensing and CAN interface"
- note removed: "Current, voltage, and temperature sensing"
- note removed: "Low-side MOSFET motor switch"
- note removed: "STM32 Nucleo, CAN, accelerometer header, and test points"
